File: KICAD/Prototypes/328PB_Breakout/328PB_Breakout.sch (KiCad schematic (older format))
At the start: 13 parts, among them SW1 SW_PUSH, U1 ATMEGA328PB, U2 AVRISP, U3 FTDI

Commit message: Added DPS310 library
Parts:
- gave numbers to parts that had none: 2
Changed lines of the file:
@@
 	3100 3200 3100 3250
 $Comp
-L RES R?
+L RES R3
 U 1 1 58758E84
 P 3100 3350
-F 0 "R?" H 3150 3275 20  0000 C CNN
+F 0 "R3" H 3150 3275 20  0000 C CNN
 F 1 "330" V 3100 3350 20  0000 C CNN
 F 2 "_Fab_Footprint:CAP_1206_FAB" H 3100 3350 60  0001 C CNN
@@
 $EndComp
 $Comp
-L GND #PWR?
+L GND #PWR010
 U 1 1 58758ECC
 P 3100 3950
-F 0 "#PWR?" H 3100 3700 60  0001 C CNN
+F 0 "#PWR010" H 3100 3700 60  0001 C CNN
 F 1 "GND" H 3100 3800 60  0000 C CNN
 F 2 "" H 3100 3950 60  0000 C CNN
@@
 $EndComp
 $Comp
-L FAB_LED L?
+L FAB_LED L2
 U 1 1 58758EFB
 P 3100 3650
-F 0 "L?" H 3200 3600 20  0000 C CNN
+F 0 "L2" H 3200 3600 20  0000 C CNN
 F 1 "FAB_LED" H 3025 3725 20  0000 C CNN
 F 2 "_Fab_Footprint:LED_1206_FAB" H 3100 3675 60  0001 C CNN
